Commit message: Issue with world

File: arv_description/urdf/arv.urdf (robot description, URDF)
Before this commit: robot arv, 9 links, 8 joints
Links:
- added link lidar_link, mass 0.15; collision cylinder length=0.0717 radius=0.0516; visual cylinder length=0.0717 radius=0.0516
Joints:
- added joint lidar_joint: type fixed, parent base_link, child lidar_link, origin xyz=0.2159 -0.02397 0.14850000000000002 rpy=0 0 0

File: arv_description/urdf/arv.urdf.xacro (robot description, xacro)
@@ -2,6 +2,6 @@
 <robot name="arv" xmlns:xacro="http://www.ros.org/wiki/xacro">
     <xacro:include filename="$(find arv_description)/urdf/arv_utils.urdf.xacro" />
-    <xacro:include filename="$(find arv_description)/urdf/sensor_plugins/arv_lidar.gazebo.xacro"/>
-    <xacro:include filename="$(find arv_description)/urdf/sensor_plugins/arv_imu.gazebo.xacro"/>
+    <xacro:include filename="$(find arv_description)/urdf/arv_lidar.gazebo.xacro"/>
+    <xacro:include filename="$(find arv_description)/urdf/arv_imu.gazebo.xacro"/>
     <xacro:property name="PI" value="3.1415926535897931"/>
     <!--    Model macros    -->
@@ -221,5 +221,5 @@
             friction_coeff="0.0" />
         <xacro:IMU base_link="${base_link_name}"/>
-        <!-- <xacro:LIDAR base_link="${base_link_name}"/> -->
+        <xacro:LIDAR base_link="${base_link_name}"/>
     </xacro:macro>
 </robot>

File: arv_description/urdf/standalone.urdf.xacro (robot description, xacro)
@@ -9,4 +9,5 @@
     <xacro:include filename="$(find arv_description)/urdf/arv.urdf.xacro"/>
     <xacro:arv />
+    <!--
     <gazebo>
         <plugin name="gazebo_ros2_control" filename="libgazebo_ros2_control.so">
@@ -15,3 +16,4 @@
         </plugin>
     </gazebo>
+    -->
 </robot>

Commit message: Model visible in gazebo
Now model is visible in both RViz2 and Gazebo. Warning: TF_OLD_DATA -> model doesn't move in Gazebo. Also topic /arv/odometry fills up.

File: arv_description/urdf/arv.urdf (robot description, URDF)
Before this commit: robot arv, 10 links, 9 joints
Joints:
- joint LEFT_FRONT_WHEEL_JOINT: axis 0 1 0 -> 0 0 1
- joint RIGHT_FRONT_WHEEL_JOINT: axis 0 1 0 -> 0 0 1

File: arv_description/urdf/arv.urdf.xacro (robot description, xacro)
@@ -12,5 +12,5 @@
             <child link="${prefix}_FRONT_WHEEL"/>
             <origin xyz="0 0 ${Y}" rpy="0 0 0" />
-            <axis xyz="0 1 0" rpy="0 0 0" />
+            <axis xyz="0 0 1" rpy="0 0 0" />
             <dynamics damping="1.0" friction="0.0"/>
             <limit effort="1" velocity="1"/>
@@ -180,18 +180,18 @@
         <!-- Fixed joint to add dummy inertia link -->
         <joint name="base_to_base_inertia" type="fixed">
-        <parent link="${base_link_name}"/>
-        <child link="base_inertia"/>
-        <origin xyz="0 0 0" rpy="0 0 0"/>
+            <parent link="${base_link_name}"/>
+            <child link="base_inertia"/>
+            <origin xyz="0 0 0" rpy="0 0 0"/>
         </joint>
         <!-- Dummy inertia link, because KDL cannot have inertia on the base link -->
         <link name="base_inertia">
-        <inertial>
-            <origin xyz="0 0 0" rpy="0 0 0"/>
-            <mass value="${chassisMass}"/>
-            <xacro:box_inertia m="${chassisMass}"
-                        x="${chassisLength}"
-                        y="${chassisWidth}"
-                        z="${chassisHeight}"/>
-        </inertial>
+            <inertial>
+                <origin xyz="0 0 0" rpy="0 0 0"/>
+                <mass value="${chassisMass}"/>
+                <xacro:box_inertia m="${chassisMass}"
+                            x="${chassisLength}"
+                            y="${chassisWidth}"
+                            z="${chassisHeight}"/>
+            </inertial>
         </link>
     </xacro:macro>

File: arv_description/urdf/arv_lidar.gazebo.xacro (robot description, xacro)
@@ -69,8 +69,5 @@
         </sensor>
       </gazebo>
-      <gazebo reference="rslidar_base_mount_joint">
-        <preserveFixedJoint>true</preserveFixedJoint>
-      </gazebo>
-      <gazebo reference="rslidar_base_scan_joint">
+      <gazebo reference="lidar_joint">
         <preserveFixedJoint>true</preserveFixedJoint>
       </gazebo>
