Commit message: IMU working

File: ack_description/urdf/arv.urdf.xacro (robot description, xacro)
@@ -1,7 +1,7 @@
 <?xml version="1.0"?>
 <robot name="arv" xmlns:xacro="http://www.ros.org/wiki/xacro">
-    <xacro:include filename="$(find arv_description)/urdf/arv_utils.urdf.xacro" />
-    <xacro:include filename="$(find arv_description)/urdf/arv_lidar.gazebo.xacro"/>
-    <xacro:include filename="$(find arv_description)/urdf/arv_imu.gazebo.xacro"/>
+    <xacro:include filename="$(find ack_description)/urdf/arv_utils.urdf.xacro" />
+    <xacro:include filename="$(find ack_description)/urdf/arv_lidar.gazebo.xacro"/>
+    <xacro:include filename="$(find ack_description)/urdf/arv_imu.gazebo.xacro"/>
     <xacro:property name="PI" value="3.1415926535897931"/>
     <!--    Model macros    -->

File: ack_description/urdf/arv_imu.gazebo.xacro (robot description, xacro)
@@ -9,5 +9,5 @@
         <xacro:property name="imu_update_rate"		value="400"/>
         <xacro:property name="imu_link"  			value="imu_link"/>
-        <xacro:property name="imu_topic" 			value="/arv/imu"/>
+        <xacro:property name="imu_topic" 			value="/imu"/>
         <xacro:property name="imu_calibration_service_name" value="/imu/calibrate"/>
         <xacro:property name="acceleration_offset"          value="0.0 0.0 0.0"/>
@@ -23,13 +23,4 @@
         <xacro:property name="heading_drift_frequency" 	value="0.0"/>
         <xacro:property name="heading_gaussian_noise" 	value="0.0"/>
-        <gazebo reference="imu_link">
-            <sensor name="imu_sensor" type="imu">
-                <always_on>1</always_on>
-                <update_rate>${imu_update_rate}</update_rate>
-                <ignition_frame_id>arv/imu_link</ignition_frame_id>
-                <visualize>true</visualize>
-                <topic>${imu_topic}</topic>
-            </sensor>
-        </gazebo>
         <!-- Imu is fixed to the base link -->
         <joint name="imu_joint" type="fixed">
@@ -57,10 +48,14 @@
                 </geometry>
             </collision>
-            <!--
-            <material name="orange">
-                <color rgba="255 108 10 255"/>
-            </material>
-            -->
         </link>
+        <gazebo reference="imu_link">
+            <sensor name="imu_sensor" type="imu">
+                <always_on>1</always_on>
+                <update_rate>${imu_update_rate}</update_rate>
+                <ignition_frame_id>arv/imu_link</ignition_frame_id>
+                <visualize>true</visualize>
+                <topic>${imu_topic}</topic>
+            </sensor>
+        </gazebo>
         <gazebo reference="${imu_link}">
             <material>Gazebo/Orange</material>

File: ack_description/urdf/arv_lidar.gazebo.xacro (robot description, xacro)
@@ -10,5 +10,5 @@
     <xacro:property name="lidar_update_rate"		value="400"/>
     <xacro:property name="lidar_link"  			value="lidar_link"/>
-    <xacro:property name="lidar_topic" 			value="/arv/scan"/>
+    <xacro:property name="lidar_topic" 			value="/scan"/>
     <joint name="lidar_joint" type="fixed">
       <origin xyz="${lidar_origin_xyz}" rpy="${lidar_origin_rpy}"/>

File: ack_description/urdf/standalone.urdf.xacro (robot description, xacro)
@@ -6,24 +6,29 @@
     <xacro:property name="lidar" value="true"/>
     <!-- Includes -->
-    <xacro:include filename="$(find arv_description)/urdf/arv_properties.urdf.xacro" />
-    <xacro:include filename="$(find arv_description)/urdf/arv.urdf.xacro"/>
-    <xacro:arv />
+    <xacro:include filename="$(find ack_description)/urdf/arv_properties.urdf.xacro" />
+    <xacro:include filename="$(find ack_description)/urdf/arv.urdf.xacro"/>
+    <xacro:arv/>
     <gazebo>
         <plugin
-            filename="ignition-gazebo-diff-drive-system"
-            name="ignition::gazebo::systems::DiffDrive">
+            filename="ignition-gazebo-ackermann-steering-system"
+            name="ignition::gazebo::systems::AckermannSteering">
             <left_joint>LEFT_FRONT_WHEEL_JOINT</left_joint>
             <right_joint>RIGHT_FRONT_WHEEL_JOINT</right_joint>
+            <left_steering_joint>LEFT_HINGE_JOINT</left_steering_joint>
+            <right_steering_joint>RIGHT_HINGE_JOINT</right_steering_joint>
             <wheel_separation>1.25</wheel_separation>
-            <wheel_radius>0.3</wheel_radius>
+            <kingpin_width>0.8</kingpin_width>
+            <wheel_base>1.0</wheel_base>
+            <steering_limit>0.5</steering_limit>
+            <wheel_radius>${wheelRadius}</wheel_radius>
             <odom_publish_frequency>1</odom_publish_frequency>
-            <max_linear_acceleration>1</max_linear_acceleration>
-            <min_linear_acceleration>-1</min_linear_acceleration>
-            <max_angular_acceleration>2</max_angular_acceleration>
-            <min_angular_acceleration>-2</min_angular_acceleration>
-            <max_linear_velocity>0.5</max_linear_velocity>
-            <min_linear_velocity>-0.5</min_linear_velocity>
-            <max_angular_velocity>1</max_angular_velocity>
-            <min_angular_velocity>-1</min_angular_velocity>
+            <min_velocity>0</min_velocity>
+            <max_velocity>10</max_velocity>
+            <min_acceleration>0</min_acceleration>
+            <max_acceleration>10</max_acceleration>
+            <min_jerk>-1</min_jerk>
+            <max_jerk>1</max_jerk>
+            <topic>arv/cmd_vel</topic>
+            <odom_topic>arv/odometry</odom_topic>
         </plugin>
     </gazebo>
