Commit message: Tuning parameters

File: ack_description/urdf/arv.urdf (robot description, URDF)
Before this commit: robot arv, 10 links, 9 joints
Links:
- link LEFT_FRONT_WHEEL: mass 5 -> 0.08; geometry collision cylinder length=0.037 radius=0.055; visual cylinder length=0.037 radius=0.055
- link LEFT_HINGE: mass 0.2 -> 0.03; geometry visual cylinder length=0.03 radius=0.01
- link LEFT_REAR_WHEEL: mass 5 -> 0.08; geometry collision cylinder length=0.037 radius=0.055; visual cylinder length=0.037 radius=0.055
- link RIGHT_FRONT_WHEEL: mass 5 -> 0.08; geometry collision cylinder length=0.037 radius=0.055; visual cylinder length=0.037 radius=0.055
- link RIGHT_HINGE: mass 0.2 -> 0.03; geometry visual cylinder length=0.03 radius=0.01
- link RIGHT_REAR_WHEEL: mass 5 -> 0.08; geometry collision cylinder length=0.037 radius=0.055; visual cylinder length=0.037 radius=0.055
- link base_inertia: mass 40 -> 2.3
- link base_link: geometry collision box size=0.57 0.29 0.075; visual box size=0.57 0.29 0.075
- link imu_link: mass 0.001 -> 0.01
Joints:
- joint LEFT_FRONT_WHEEL_JOINT: origin xyz=0 0 0.09 rpy=0 0 0 -> xyz=0 0 0.0335 rpy=0 0 0
- joint LEFT_HINGE_JOINT: axis 0 1 0 -> 0 -1 0; limit lower=-1 upper=1 effort=100 velocity=1 -> lower=-0.53 upper=0.53 effort=100 velocity=1; origin xyz=0.2159 0.255 -0.018500000000000003 rpy=-1.5707963267948966 0.0 0.0 -> xyz=0.162 0.15999999999999998 -0.0295 rpy=-1.5707963267948966 0.0 0.0
- joint LEFT_REAR_WHEEL_JOINT: axis 0 0 1 -> 0 0 -1; origin xyz=-0.2159 0.345 -0.018500000000000003 rpy=1.5707963267948966 0 0 -> xyz=-0.162 0.1735 -0.0295 rpy=1.5707963267948966 0 0
- joint RIGHT_FRONT_WHEEL_JOINT: origin xyz=0 0 -0.09 rpy=0 0 0 -> xyz=0 0 -0.0335 rpy=0 0 0
- joint RIGHT_HINGE_JOINT: axis 0 1 0 -> 0 -1 0; limit lower=-1 upper=1 effort=100 velocity=1 -> lower=-0.53 upper=0.53 effort=100 velocity=1; origin xyz=0.2159 -0.255 -0.018500000000000003 rpy=-1.5707963267948966 0.0 0.0 -> xyz=0.162 -0.15999999999999998 -0.0295 rpy=-1.5707963267948966 0.0 0.0
- joint RIGHT_REAR_WHEEL_JOINT: axis 0 0 1 -> 0 0 -1; origin xyz=-0.2159 -0.345 -0.018500000000000003 rpy=1.5707963267948966 0 0 -> xyz=-0.162 -0.1735 -0.0295 rpy=1.5707963267948966 0 0
- joint imu_joint: origin xyz=-0.2159 -0.02397 0.10350000000000001 rpy=0 0 0 -> xyz=-0.162 0 0.042499999999999996 rpy=0 0 0
- joint lidar_joint: origin xyz=0.2159 -0.02397 0.14850000000000002 rpy=0 0 0 -> xyz=0.162 0 0.0875 rpy=0 0 0

File: ack_description/urdf/arv.urdf.xacro (robot description, xacro)
@@ -63,7 +63,7 @@
             <child link="${prefix}_HINGE"/>
             <origin xyz="${X} ${Y} ${wheelHeight - chassisHeight/2.0}" rpy="-${0.5*PI} 0.0 0.0"/>
-            <axis xyz="0 1 0" rpy="0 0 0"/>
+            <axis xyz="0 -1 0" rpy="0 0 0"/>
             <dynamics damping="0.0" friction="0.0"/>
-            <limit lower="-1" upper="1" effort="100" velocity="1"/>
+            <limit lower="-0.53" upper="0.53" effort="100" velocity="1"/>
         </joint>
         <link name="${prefix}_HINGE">
@@ -111,5 +111,5 @@
             <child link="${prefix}_REAR_WHEEL"/>
             <origin xyz="${X} ${Y} ${wheelHeight - chassisHeight/2.0}" rpy="${PI/2} 0 0" />
-            <axis xyz="0 0 1" rpy="0 0 0" />
+            <axis xyz="0 0 -1" rpy="0 0 0" />
             <dynamics damping="1.0" friction="0.0"/>
             <limit effort="1" velocity="1"/>

File: ack_description/urdf/arv_imu.gazebo.xacro (robot description, xacro)
@@ -6,5 +6,5 @@
         <xacro:property name="imu_base_link"		value="${base_link}"/>
         <xacro:property name="imu_origin_rpy"		value="0 0 0"/>
-        <xacro:property name="imu_origin_xyz"		value="-0.2159 -0.02397 ${chassisHeight/2.0+0.005}"/>
+        <xacro:property name="imu_origin_xyz"		value="${backWheelX} 0 ${chassisHeight/2.0+0.005}"/>
         <xacro:property name="imu_update_rate"		value="400"/>
         <xacro:property name="imu_link"  			value="imu_link"/>
@@ -32,5 +32,5 @@
         <link name="${imu_link}">
             <inertial>
-                <mass value="0.001"/>
+                <mass value="0.01"/>
                 <origin rpy="0 0 0" xyz="0 0 0"/>
                 <inertia ixx="0.0001" ixy="0" ixz="0" iyy="0.000001" iyz="0" izz="0.0001"/>

File: ack_description/urdf/arv_lidar.gazebo.xacro (robot description, xacro)
@@ -4,5 +4,5 @@
     <xacro:property name="lidar_base_link"		value="${base_link}"/>
     <xacro:property name="lidar_origin_rpy"		value="0 0 0"/>
-    <xacro:property name="lidar_origin_xyz"		value="${hingeX} -0.02397 ${chassisHeight/2.0+0.05}"/>
+    <xacro:property name="lidar_origin_xyz"		value="${hingeX} 0 ${chassisHeight/2.0+0.05}"/>
     <xacro:property name="lidar_height"		value="0.0717"/>
     <xacro:property name="lidar_radius"		value="0.0516"/>

File: ack_description/urdf/arv_properties.urdf.xacro (robot description, xacro)
@@ -2,17 +2,17 @@
 <robot xmlns:xacro="http://www.ros.org/wiki/xacro" name="arv">
     <xacro:property name="base_link_name" value="base_link"/>
-    <xacro:property name="chassisHeight" value="0.197"/>
-    <xacro:property name="chassisLength" value="0.605"/>
-    <xacro:property name="chassisWidth" value="0.410"/>
-    <xacro:property name="chassisMass" value="40"/>
-    <xacro:property name="hingeMass" value="0.2"/>
-    <xacro:property name="hingeRadius" value="0.06"/>
-    <xacro:property name="hingeLength" value="0.1"/>
-    <xacro:property name="hingeX" value="0.2159"/>
-    <xacro:property name="wheelWidth" value="0.08"/>
-    <xacro:property name="wheelRadius" value="0.15"/>
-    <xacro:property name="backWheelX" value="-0.2159"/>
-    <xacro:property name="wheelClearance" value="0.1"/>
-    <xacro:property name="wheelHeight" value="0.08"/>
-    <xacro:property name="wheelMass" value="5"/>
+    <xacro:property name="chassisHeight" value="0.075"/>
+    <xacro:property name="chassisLength" value="0.570"/>
+    <xacro:property name="chassisWidth" value="0.290"/>
+    <xacro:property name="chassisMass" value="2.300"/>
+    <xacro:property name="hingeMass" value="0.030"/>
+    <xacro:property name="hingeRadius" value="0.010"/>
+    <xacro:property name="hingeLength" value="0.030"/>
+    <xacro:property name="hingeX" value="0.162"/>
+    <xacro:property name="wheelWidth" value="0.037"/>
+    <xacro:property name="wheelRadius" value="0.055"/>
+    <xacro:property name="backWheelX" value="-0.162"/>
+    <xacro:property name="wheelClearance" value="0.01"/>
+    <xacro:property name="wheelHeight" value="0.008"/>
+    <xacro:property name="wheelMass" value="0.08"/>
 </robot>

File: ack_description/urdf/standalone.urdf.xacro (robot description, xacro)
@@ -19,20 +19,16 @@
             <left_steering_joint>LEFT_HINGE_JOINT</left_steering_joint>
             <right_steering_joint>RIGHT_HINGE_JOINT</right_steering_joint>
-            <wheel_separation>1.25</wheel_separation>
-            <kingpin_width>0.8</kingpin_width>
-            <wheel_base>1.0</wheel_base>
+            <wheel_separation>0.47</wheel_separation>
+            <kingpin_width>0.47</kingpin_width>
+            <wheel_base>0.324</wheel_base>
             <steering_limit>0.5</steering_limit>
             <wheel_radius>0.15</wheel_radius>
             <odom_publish_frequency>1</odom_publish_frequency>
-            <min_velocity>-1</min_velocity>
+            <min_velocity>-10</min_velocity>
             <max_velocity>10</max_velocity>
-            <min_acceleration>-3</min_acceleration>
+            <min_acceleration>-10</min_acceleration>
             <max_acceleration>10</max_acceleration>
-            <!--
-            <min_jerk>-1</min_jerk>
-            <max_jerk>1</max_jerk>
-            <topic>arv/cmd_vel</topic>
-            <odom_topic>arv/odometry</odom_topic>
-            -->
+            <min_jerk>-10</min_jerk>
+            <max_jerk>10</max_jerk>
         </plugin>
     </gazebo>

Commit message: Model can be driven. Drifting is an issue

File: ack_description/urdf/arv.urdf (robot description, URDF)
Before this commit: robot arv, 10 links, 9 joints
Joints:
- joint LEFT_FRONT_WHEEL_JOINT: limit effort=1 velocity=1 -> effort=100 velocity=200
- joint LEFT_REAR_WHEEL_JOINT: limit effort=1 velocity=1 -> effort=100 velocity=200
- joint RIGHT_FRONT_WHEEL_JOINT: limit effort=1 velocity=1 -> effort=100 velocity=200
- joint RIGHT_REAR_WHEEL_JOINT: limit effort=1 velocity=1 -> effort=100 velocity=200

File: ack_description/urdf/arv.urdf.xacro (robot description, xacro)
@@ -7,5 +7,5 @@
     <!--    Model macros    -->
     <!-- Front Wheel -->
-    <xacro:macro name="front_wheel" params="prefix X Y friction_coeff:=0.2 transmission_reduction:=1" >
+    <xacro:macro name="front_wheel" params="prefix X Y friction_coeff:=0.7 transmission_reduction:=1" >
         <joint name="${prefix}_FRONT_WHEEL_JOINT" type="continuous">
             <parent link="${prefix}_HINGE"/>
@@ -13,6 +13,6 @@
             <origin xyz="0 0 ${Y}" rpy="0 0 0" />
             <axis xyz="0 0 1" rpy="0 0 0" />
-            <dynamics damping="1.0" friction="0.0"/>
-            <limit effort="1" velocity="1"/>
+            <dynamics damping="0.0" friction="0.0"/>
+            <limit effort="100" velocity="200"/>
             <joint_properties damping="0.2" friction="0.2"/>
         </joint>
@@ -58,5 +58,5 @@
     </xacro:macro>
     <!-- Front Hinge -->
-    <xacro:macro name="hinge" params="prefix X Y friction_coeff:=0.2 transmission_reduction:=1">
+    <xacro:macro name="hinge" params="prefix X Y">
         <joint name="${prefix}_HINGE_JOINT" type="revolute">
             <parent link="${base_link_name}"/>
@@ -87,6 +87,6 @@
         </link>
         <gazebo reference="${prefix}_WHEEL_HINGE">
-            <mu1 value="${friction_coeff}"/>
-            <mu2 value="${friction_coeff}"/>
+            <mu1 value="0.0"/>
+            <mu2 value="0.0"/>
             <kp>10000000.0</kp>
             <kd>1.0</kd>
@@ -101,10 +101,10 @@
             <actuator name="${prefix}_ACTUATOR">
                 <hardwareInterface>EffortJointInterface</hardwareInterface>
-                <mechanicalReduction>${transmission_reduction}</mechanicalReduction>
+                <mechanicalReduction>1</mechanicalReduction>
             </actuator>
         </transmission>
     </xacro:macro>
     <!-- Rear Wheel -->
-    <xacro:macro name="rear_wheel" params="prefix X Y friction_coeff:=0.2 transmission_reduction:=1" >
+    <xacro:macro name="rear_wheel" params="prefix X Y friction_coeff:=0.7 transmission_reduction:=1" >
         <joint name="${prefix}_REAR_WHEEL_JOINT" type="continuous">
             <parent link="${base_link_name}"/>
@@ -112,6 +112,6 @@
             <origin xyz="${X} ${Y} ${wheelHeight - chassisHeight/2.0}" rpy="${PI/2} 0 0" />
             <axis xyz="0 0 -1" rpy="0 0 0" />
-            <dynamics damping="1.0" friction="0.0"/>
-            <limit effort="1" velocity="1"/>
+            <dynamics damping="0.0" friction="0.0"/>
+            <limit effort="100" velocity="200"/>
             <joint_properties damping="0.2" friction="0.2"/>
         </joint>
@@ -196,5 +196,5 @@
         </link>
     </xacro:macro>
-    <xacro:macro name="arv" params="wheel_joint_type:=continuous lidar:=true simulation:=true">
+    <xacro:macro name="arv">
         <xacro:chassis/>
         <xacro:hinge prefix="LEFT"

File: ack_description/urdf/standalone.urdf.xacro (robot description, xacro)
@@ -9,27 +9,3 @@
     <xacro:include filename="$(find ack_description)/urdf/arv.urdf.xacro"/>
     <xacro:arv/>
-    <gazebo>
-        <plugin
-            filename="ignition-gazebo-ackermann-steering-system"
-            name="ignition::gazebo::systems::AckermannSteering">
-            <left_joint>LEFT_FRONT_WHEEL_JOINT</left_joint>
-            <left_joint>LEFT_REAR_WHEEL_JOINT</left_joint>
-            <right_joint>RIGHT_FRONT_WHEEL_JOINT</right_joint>
-            <right_joint>RIGHT_REAR_WHEEL_JOINT</right_joint>
-            <left_steering_joint>LEFT_HINGE_JOINT</left_steering_joint>
-            <right_steering_joint>RIGHT_HINGE_JOINT</right_steering_joint>
-            <wheel_separation>0.47</wheel_separation>
-            <kingpin_width>0.47</kingpin_width>
-            <wheel_base>0.324</wheel_base>
-            <steering_limit>0.5</steering_limit>
-            <wheel_radius>0.15</wheel_radius>
-            <odom_publish_frequency>1</odom_publish_frequency>
-            <min_velocity>-10</min_velocity>
-            <max_velocity>10</max_velocity>
-            <min_acceleration>-10</min_acceleration>
-            <max_acceleration>10</max_acceleration>
-            <min_jerk>-10</min_jerk>
-            <max_jerk>10</max_jerk>
-        </plugin>
-    </gazebo>
 </robot>
