Commit message: Import improvements from ARS project

File: ars_description/urdf/arc.urdf (robot description, URDF)
Before this commit: robot arc, 10 links, 9 joints
Links:
- removed link base_inertia
- added link chassis, mass 2.3; collision box size=0.57 0.29 0.075; visual box size=0.57 0.29 0.075
- link LEFT_FRONT_WHEEL: geometry collision sphere radius=0.055; visual cylinder length=0.037 radius=0.055
- link LEFT_REAR_WHEEL: geometry collision sphere radius=0.055; visual cylinder length=0.037 radius=0.055
- link RIGHT_FRONT_WHEEL: geometry collision sphere radius=0.055; visual cylinder length=0.037 radius=0.055
- link RIGHT_REAR_WHEEL: geometry collision sphere radius=0.055; visual cylinder length=0.037 radius=0.055
- link base_link: geometry 
Joints:
- removed joint base_to_base_inertia
- added joint chassis_joinz: type fixed, parent base_link, child chassis, origin xyz=0 0 0.08449999999999999 rpy=0 0 0
- joint LEFT_FRONT_WHEEL_JOINT: limit effort=100 velocity=200 -> (none)
- joint LEFT_HINGE_JOINT: limit lower=-0.53 upper=0.53 effort=100 velocity=1 -> (none); parent base_link -> chassis; type revolute -> continuous
- joint LEFT_REAR_WHEEL_JOINT: limit effort=100 velocity=200 -> (none); origin xyz=-0.162 0.1735 -0.0295 rpy=1.5707963267948966 0 0 -> xyz=-0.162 0.19349999999999998 -0.0295 rpy=1.5707963267948966 0 0; parent base_link -> chassis
- joint RIGHT_FRONT_WHEEL_JOINT: limit effort=100 velocity=200 -> (none)
- joint RIGHT_HINGE_JOINT: limit lower=-0.53 upper=0.53 effort=100 velocity=1 -> (none); parent base_link -> chassis; type revolute -> continuous
- joint RIGHT_REAR_WHEEL_JOINT: limit effort=100 velocity=200 -> (none); origin xyz=-0.162 -0.1735 -0.0295 rpy=1.5707963267948966 0 0 -> xyz=-0.162 -0.19349999999999998 -0.0295 rpy=1.5707963267948966 0 0; parent base_link -> chassis
- joint imu_joint: parent base_link -> chassis
- joint lidar_joint: parent base_link -> chassis

File: ars_description/urdf/arc.xacro (robot description, xacro)
@@ -10,6 +10,5 @@
     <xacro:include filename="$(find ars_description)/urdf/sensors/imu.xacro"/>
     <xacro:include filename="$(find ars_description)/urdf/sensors/lidar.xacro"/>
-    <!--<xacro:include filename="$(find ars_description)/urdf/transmissions.xacro"/>-->
-    <xacro:include filename="$(find ars_description)/urdf/gazebo.xacro"/>
+    <xacro:include filename="$(find ars_description)/urdf/ros2_control.xacro"/>
     <xacro:chassis/>
     <xacro:hinge prefix="LEFT"
@@ -27,8 +26,8 @@
     <xacro:rear_wheel prefix="LEFT"
         X="${backWheelX}"
-        Y="${chassisWidth/2+wheelClearance+wheelWidth/2}"/>
+        Y="${chassisWidth/2+hingeLength+wheelWidth/2}"/>
     <xacro:rear_wheel prefix="RIGHT"
         X="${backWheelX}"
-        Y="${-chassisWidth/2-wheelClearance-wheelWidth/2}"/>
+        Y="${-chassisWidth/2-hingeLength-wheelWidth/2}"/>
     <xacro:IMU base_link="${base_link_name}"/>
     <xacro:LIDAR base_link="${base_link_name}"/>

File: ars_description/urdf/parts/chassis.xacro (robot description, xacro)
@@ -2,5 +2,6 @@
 <robot xmlns:xacro="http://www.ros.org/wiki/xacro">
     <xacro:macro name="chassis">
-        <link name="${base_link_name}">
+        <link name="base_link"/>
+        <link name="chassis">
             <collision>
                 <origin xyz="0 0 0" rpy="0 0 0"/>
@@ -18,13 +19,4 @@
                 </material>
             </visual>
-        </link>
-        <!-- Fixed joint to add dummy inertia link -->
-        <joint name="base_to_base_inertia" type="fixed">
-            <parent link="${base_link_name}"/>
-            <child link="base_inertia"/>
-            <origin xyz="0 0 0" rpy="0 0 0"/>
-        </joint>
-        <!-- Dummy inertia link, because KDL cannot have inertia on the base link -->
-        <link name="base_inertia">
             <inertial>
                 <origin xyz="0 0 0" rpy="0 0 0"/>
@@ -38,4 +30,10 @@
             </inertial>
         </link>
+        <!-- Fixed joint to add dummy inertia link -->
+        <joint name="chassis_joinz" type="fixed">
+            <parent link="base_link"/>
+            <child link="chassis"/>
+            <origin xyz="0 0 ${wheelRadius - wheelHeight + chassisHeight/2.0}" rpy="0 0 0"/>
+        </joint>
     </xacro:macro>
 </robot>

File: ars_description/urdf/parts/front_wheel.xacro (robot description, xacro)
@@ -7,7 +7,5 @@
             <origin xyz="0 0 ${Y}" rpy="0 0 0" />
             <axis xyz="0 0 1" rpy="0 0 0" />
-            <dynamics damping="0.0" friction="0.0"/>
-            <limit effort="100" velocity="200"/>
-            <joint_properties damping="0.2" friction="0.2"/>
+            <dynamics damping="0.2"/>
         </joint>
         <link name="${prefix}_FRONT_WHEEL">
@@ -15,5 +13,5 @@
                 <origin xyz="0 0 0" rpy="0 0 0" />
                 <geometry>
-                    <cylinder length="${wheelWidth}" radius="${wheelRadius}"/>
+                    <sphere radius="${wheelRadius}"/>
                 </geometry>
             </collision>

File: ars_description/urdf/parts/hinge.xacro (robot description, xacro)
@@ -2,11 +2,9 @@
 <robot xmlns:xacro="http://www.ros.org/wiki/xacro">
     <xacro:macro name="hinge" params="prefix X Y">
-        <joint name="${prefix}_HINGE_JOINT" type="revolute">
-            <parent link="${base_link_name}"/>
+        <joint name="${prefix}_HINGE_JOINT" type="continuous">
+            <parent link="chassis"/>
             <child link="${prefix}_HINGE"/>
             <origin xyz="${X} ${Y} ${wheelHeight - chassisHeight/2.0}" rpy="-${0.5*PI} 0.0 0.0"/>
             <axis xyz="0 -1 0" rpy="0 0 0"/>
-            <dynamics damping="0.0" friction="0.0"/>
-            <limit lower="-0.53" upper="0.53" effort="100.0" velocity="5.0"/>
         </joint>
         <link name="${prefix}_HINGE">

File: ars_description/urdf/parts/rear_wheel.xacro (robot description, xacro)
@@ -3,11 +3,8 @@
     <xacro:macro name="rear_wheel" params="prefix X Y friction_coeff:=0.7 transmission_reduction:=1" >
         <joint name="${prefix}_REAR_WHEEL_JOINT" type="continuous">
-            <parent link="${base_link_name}"/>
+            <parent link="chassis"/>
             <child link="${prefix}_REAR_WHEEL"/>
             <origin xyz="${X} ${Y} ${wheelHeight - chassisHeight/2.0}" rpy="${PI/2} 0 0" />
             <axis xyz="0 0 -1" rpy="0 0 0" />
-            <dynamics damping="0.0" friction="0.0"/>
-            <limit effort="100" velocity="200"/>
-            <joint_properties damping="0.2" friction="0.2"/>
         </joint>
         <link name="${prefix}_REAR_WHEEL">
@@ -15,5 +12,5 @@
                 <origin xyz="0 0 0" rpy="0 0 0" />
                 <geometry>
-                    <cylinder length="${wheelWidth}" radius="${wheelRadius}"/>
+                    <sphere radius="${wheelRadius}"/>
                 </geometry>
             </collision>

File: ars_description/urdf/sensors/imu.xacro (robot description, xacro)
@@ -5,5 +5,5 @@
         <joint name="imu_joint" type="fixed">
             <origin xyz="${imu_origin_xyz}" rpy="${imu_origin_rpy}"/>
-            <parent link="${base_link}"/>
+            <parent link="chassis"/>
             <child link="imu_link"/>
         </joint>
@@ -28,4 +28,16 @@
             </collision>
         </link>
+        <gazebo reference="imu_link">
+            <sensor name="imu_sensor" type="imu">
+                <always_on>1</always_on>
+                <update_rate>${imu_update_rate}</update_rate>
+                <ignition_frame_id>imu_link</ignition_frame_id>
+                <visualize>true</visualize>
+                <topic>${imu_topic}</topic>
+            </sensor>
+        </gazebo>
+        <!-- <gazebo reference="imu_joint">
+            <preserveFixedJoint>true</preserveFixedJoint>
+        </gazebo> -->
     </xacro:macro>
 </robot>

File: ars_description/urdf/sensors/lidar.xacro (robot description, xacro)
@@ -5,5 +5,5 @@
         <joint name="lidar_joint" type="fixed">
             <origin xyz="${lidar_origin_xyz}" rpy="${lidar_origin_rpy}"/>
-            <parent link="${base_link}"/>
+            <parent link="chassis"/>
             <child link="lidar_link"/>
         </joint>
@@ -28,4 +28,42 @@
             </collision>
         </link>
+        <gazebo reference="lidar_link">
+            <sensor name='gpu_lidar' type='gpu_lidar'>
+                <topic>${lidar_topic}</topic>
+                <update_rate>${lidar_update_rate}</update_rate>
+                <alwaysOn>1</alwaysOn>
+                <visualize>true</visualize>
+                <ignition_frame_id>lidar_link</ignition_frame_id>
+                <lidar>
+                    <scan>
+                        <horizontal>
+                            <samples>640</samples>
+                            <resolution>1</resolution>
+                            <min_angle>-1.396263</min_angle>
+                            <max_angle>1.396263</max_angle>
+                        </horizontal>
+                        <vertical>
+                        <samples>1</samples>
+                        <resolution>1</resolution>
+                        <min_angle>0.0</min_angle>
+                        <max_angle>0.0</max_angle>
+                        </vertical>
+                    </scan>
+                    <range>
+                        <min>0.08</min>
+                        <max>10</max>
+                        <resolution>0.01</resolution>
+                    </range>
+                    <noise>
+                        <type>gaussian</type>
+                        <mean>0.0</mean>
+                        <stddev>0.001</stddev>
+                    </noise>
+                </lidar>
+            </sensor>
+        </gazebo>
+        <!-- <gazebo reference="lidar_joint">
+            <preserveFixedJoint>true</preserveFixedJoint>
+        </gazebo> -->
     </xacro:macro>
 </robot>
